File: hardware/stm32pcb/stm32pcb.kicad_sch (KiCad schematic)
At the start: 23 parts, among them J1 Conn_02x07_Odd_Even, J2 Conn_01x02, J3 Conn_01x02, J4 Conn_01x02, U1 STM32L021K4Tx, U2 MCP4801-E/SN, U3 BU33SD5WG-TR

Commit message: add Empreintes
Parts:
- C1, C2, C3, C4, C5, C6, C9: footprint (none) -> Capacitor_SMD:C_0805_2012Metric_Pad1.18x1.45mm_HandSolder
- C10, C7, C8: footprint (none) -> Capacitor_SMD:C_0805_2012Metric
- D1, D2: footprint (none) -> LED_SMD:LED_0603_1608Metric_Pad1.05x0.95mm_HandSolder
- J1: footprint (none) -> Connector_PinHeader_1.27mm:PinHeader_2x07_P1.27mm_Vertical_SMD
- J2: value Conn_01x02 -> INPUT; footprint (none) -> Connector_JST:JST_XH_B2B-XH-A_1x02_P2.50mm_Vertical
- J3: value Conn_01x02 -> POWER; footprint (none) -> Connector_JST:JST_XH_B2B-XH-A_1x02_P2.50mm_Vertical
- J4: value Conn_01x02 -> OUTPUT; footprint (none) -> Connector_JST:JST_XH_B2B-XH-A_1x02_P2.50mm_Vertical
- L1: footprint (none) -> Inductor_SMD:L_0805_2012Metric_Pad1.05x1.20mm_HandSolder
- R1, R2, R3: footprint (none) -> Resistor_SMD:R_0805_2012Metric_Pad1.20x1.40mm_HandSolder
- U2: footprint (none) -> Package_SO:SOIC-8_3.9x4.9mm_P1.27mm

Commit message: Routage fini
Parts:
- added H1, H2, H3, H4: MountingHole_Pad, MountingHole:MountingHole_3.2mm_M3_Pad, symbol Mechanical:MountingHole_Pad
Connections:
- net GND: now also H1.1, H2.1, H3.1, H4.1
- no-connect marks 0 -> 20
Other:
- note added: "Mounting Holes"
